Commit message: URDF reworked

File: urdf/pupper_ros.urdf (robot description, URDF)
Before this commit: robot pupper_ros, 5 links, 4 joints
Links:
- added link forearm_b_l; visual box size=0.2 0.05 0.03
- added link forearm_b_r; visual box size=0.2 0.05 0.03
- added link forearm_f_l; visual box size=0.2 0.05 0.03
- added link forearm_f_r; visual box size=0.2 0.05 0.03
- added link leg_b_l_knee; visual sphere radius=0.04
- added link leg_b_r_knee; visual sphere radius=0.04
- added link leg_f_l_knee; visual sphere radius=0.04
- added link leg_f_r_knee; visual sphere radius=0.04
- added link shldr_b_l; visual sphere radius=0.06
- added link shldr_b_r; visual sphere radius=0.06
- added link shldr_f_l; visual sphere radius=0.06
- added link shldr_f_r; visual sphere radius=0.06
- link leg_b_l: geometry visual box size=0.2 0.05 0.03
- link leg_b_r: geometry visual box size=0.2 0.05 0.03
- link leg_f_l: geometry visual box size=0.2 0.05 0.03
- link leg_f_r: geometry visual box size=0.2 0.05 0.03
- link torso: geometry visual box size=0.6 0.2 0.15
Joints:
- added joint forearm_b_l_joint: type continuous, parent shldr_b_l, child forearm_b_l, origin xyz=0 0 0 rpy=0 0 0, axis 0 1 0
- added joint forearm_b_r_joint: type continuous, parent shldr_b_r, child forearm_b_r, origin xyz=0 0 0 rpy=0 0 0, axis 0 1 0
- added joint forearm_f_l_joint: type continuous, parent shldr_f_l, child forearm_f_l, origin xyz=0 0 0 rpy=0 0 0, axis 0 1 0
- added joint forearm_f_r_joint: type continuous, parent shldr_f_r, child forearm_f_r, origin xyz=0 0 0 rpy=0 0 0, axis 0 1 0
- added joint leg_b_l_knee_joint: type fixed, parent leg_b_l_knee, child leg_b_l, origin xyz=0 0 0 rpy=0 0 0, axis 0 1 0
- added joint leg_b_r_knee_joint: type fixed, parent leg_b_r_knee, child leg_b_r, origin xyz=0 0 0 rpy=0 0 0, axis 0 1 0
- added joint leg_f_l_knee_joint: type fixed, parent leg_f_l_knee, child leg_f_l, origin xyz=0 0 0 rpy=0 0 0, axis 0 1 0
- added joint leg_f_r_knee_joint: type fixed, parent leg_f_r_knee, child leg_f_r, origin xyz=0 0 0 rpy=0 0 0, axis 0 1 0
- added joint shldr_b_l_joint: type continuous, parent torso, child shldr_b_l, origin xyz=-0.32 0.15 0.4 rpy=1.57 0.0 0.0, axis 0 0 1
- added joint shldr_b_r_joint: type continuous, parent torso, child shldr_b_r, origin xyz=-0.32 -0.15 0.4 rpy=1.57 0.0 0.0, axis 0 0 1
- added joint shldr_f_l_joint: type continuous, parent torso, child shldr_f_l, origin xyz=0.32 0.15 0.4 rpy=1.57 0.0 0.0, axis 0 0 1
- added joint shldr_f_r_joint: type continuous, parent torso, child shldr_f_r, origin xyz=0.32 -0.15 0.4 rpy=1.57 0.0 0.0, axis 0 0 1
- joint leg_b_l_joint: child leg_b_l -> leg_b_l_knee; origin xyz=-0.1 0.05 0.0 rpy=0.0 0.0 0.0 -> xyz=0 -0.23 0 rpy=0 0 0; parent torso -> forearm_b_l
- joint leg_b_r_joint: child leg_b_r -> leg_b_r_knee; origin xyz=-0.1 -0.05 0.0 rpy=0.0 0.0 0.0 -> xyz=0 -0.23 0 rpy=0 0 0; parent torso -> forearm_b_r
- joint leg_f_l_joint: child leg_f_l -> leg_f_l_knee; origin xyz=0.1 0.05 0.0 rpy=0.0 0.0 0.0 -> xyz=0 -0.23 0 rpy=0 0 0; parent torso -> forearm_f_l
- joint leg_f_r_joint: child leg_f_r -> leg_f_r_knee; origin xyz=0.1 -0.05 0.0 rpy=0.0 0.0 0.0 -> xyz=0 -0.23 0 rpy=0 0 0; parent torso -> forearm_f_r

Commit message: Update pupper_ros.urdf
original dog dimetions updated to urdf

File: urdf/pupper_ros.urdf (robot description, URDF)
Before this commit: robot pupper_ros, 17 links, 16 joints
Links:
- removed link shldr_b_l
- removed link shldr_b_r
- removed link shldr_f_l
- removed link shldr_f_r
- added link leg_b_l_foot; visual sphere radius=0.04
- added link leg_b_r_foot; visual sphere radius=0.04
- added link leg_f_l_foot; visual sphere radius=0.04
- added link leg_f_r_foot; visual sphere radius=0.04
- added link shldr_b_l_1; visual cylinder length=0.1 radius=0.05
- added link shldr_b_l_2; visual cylinder length=0.066 radius=0.05
- added link shldr_b_r_1; visual cylinder length=0.1 radius=0.05
- added link shldr_b_r_2; visual cylinder length=0.066 radius=0.05
- added link shldr_f_l_1; visual cylinder length=0.1 radius=0.05
- added link shldr_f_l_2; visual cylinder length=0.066 radius=0.05
- added link shldr_f_r_1; visual cylinder length=0.1 radius=0.05
- added link shldr_f_r_2; visual cylinder length=0.066 radius=0.05
- link forearm_b_l: geometry visual box size=0.202 0.05 0.03
- link forearm_b_r: geometry visual box size=0.202 0.05 0.03
- link forearm_f_l: geometry visual box size=0.202 0.05 0.03
- link forearm_f_r: geometry visual box size=0.202 0.05 0.03
- link leg_b_l: geometry visual box size=0.177 0.05 0.03
- link leg_b_l_knee: geometry visual cylinder length=0.066 radius=0.05
- link leg_b_r: geometry visual box size=0.177 0.05 0.03
- link leg_b_r_knee: geometry visual cylinder length=0.066 radius=0.05
- link leg_f_l: geometry visual box size=0.177 0.05 0.03
- link leg_f_l_knee: geometry visual cylinder length=0.066 radius=0.05
- link leg_f_r: geometry visual box size=0.177 0.05 0.03
- link leg_f_r_knee: geometry visual cylinder length=0.066 radius=0.05
- link torso: geometry visual box size=0.26 0.26 0.15
Joints:
- added joint leg_b_l_foot_joint: type fixed, parent leg_b_l, child leg_b_l_foot, origin xyz=0 -0.197 0 rpy=0 0 0, axis 0 0 0
- added joint leg_b_r_foot_joint: type fixed, parent leg_b_r, child leg_b_r_foot, origin xyz=0 -0.197 0 rpy=0 0 0, axis 0 0 0
- added joint leg_f_l_foot_joint: type fixed, parent leg_f_l, child leg_f_l_foot, origin xyz=0 -0.197 0 rpy=0 0 0, axis 0 0 0
- added joint leg_f_r_foot_joint: type fixed, parent leg_f_r, child leg_f_r_foot, origin xyz=0 -0.197 0 rpy=0 0 0, axis 0 0 0
- added joint shldr_b_l_joint_inter: type fixed, parent shldr_b_l_1, child shldr_b_l_2, origin xyz=0 0.06 -0.1 rpy=0 1.57 1.57, axis 0 0 1
- added joint shldr_b_r_joint_inter: type fixed, parent shldr_b_r_1, child shldr_b_r_2, origin xyz=0 -0.06 -0.1 rpy=0 1.57 1.57, axis 0 0 1
- added joint shldr_f_l_joint_inter: type fixed, parent shldr_f_l_1, child shldr_f_l_2, origin xyz=0 0.06 0.1 rpy=0 1.57 1.57, axis 0 0 1
- added joint shldr_f_r_joint_inter: type fixed, parent shldr_f_r_1, child shldr_f_r_2, origin xyz=0 -0.06 0.1 rpy=0 1.57 1.57, axis 0 0 1
- joint forearm_b_l_joint: parent shldr_b_l -> shldr_b_l_2
- joint forearm_b_r_joint: parent shldr_b_r -> shldr_b_r_2
- joint forearm_f_l_joint: parent shldr_f_l -> shldr_f_l_2
- joint forearm_f_r_joint: parent shldr_f_r -> shldr_f_r_2
- joint shldr_b_l_joint: child shldr_b_l -> shldr_b_l_1; origin xyz=-0.32 0.15 0.4 rpy=1.57 0.0 0.0 -> xyz=-0.18 0.1 0.4 rpy=0 1.57 0
- joint shldr_b_r_joint: child shldr_b_r -> shldr_b_r_1; origin xyz=-0.32 -0.15 0.4 rpy=1.57 0.0 0.0 -> xyz=-0.18 -0.1 0.4 rpy=0 1.57 0
- joint shldr_f_l_joint: child shldr_f_l -> shldr_f_l_1; origin xyz=0.32 0.15 0.4 rpy=1.57 0.0 0.0 -> xyz=0.18 0.1 0.4 rpy=0 1.57 0
- joint shldr_f_r_joint: child shldr_f_r -> shldr_f_r_1; origin xyz=0.32 -0.15 0.4 rpy=1.57 0.0 0.0 -> xyz=0.18 -0.1 0.4 rpy=0 1.57 0

Commit message: looks like it works

File: urdf/pupper_ros.urdf (robot description, URDF)
Before this commit: robot pupper_ros, 25 links, 24 joints
Joints:
- joint forearm_b_l_joint: type continuous -> fixed
- joint forearm_b_r_joint: type continuous -> fixed
- joint forearm_f_l_joint: type continuous -> fixed
- joint forearm_f_r_joint: type continuous -> fixed
- joint leg_b_l_joint: axis 0 1 0 -> 0 0 1; origin xyz=0 -0.23 0 rpy=0 0 0 -> xyz=0 -0.23 0 rpy=0 0 1
- joint leg_b_l_knee_joint: axis 0 1 0 -> 0 0 1
- joint leg_b_r_joint: axis 0 1 0 -> 0 0 1; origin xyz=0 -0.23 0 rpy=0 0 0 -> xyz=0 -0.23 0 rpy=0 0 1
- joint leg_b_r_knee_joint: axis 0 1 0 -> 0 0 1
- joint leg_f_l_joint: axis 0 1 0 -> 0 0 1; origin xyz=0 -0.23 0 rpy=0 0 0 -> xyz=0 -0.23 0 rpy=0 0 1
- joint leg_f_l_knee_joint: axis 0 1 0 -> 0 0 1
- joint leg_f_r_joint: axis 0 1 0 -> 0 0 1; origin xyz=0 -0.23 0 rpy=0 0 0 -> xyz=0 -0.23 0 rpy=0 0 1
- joint leg_f_r_knee_joint: axis 0 1 0 -> 0 0 1
- joint shldr_b_l_joint_inter: type fixed -> continuous
- joint shldr_b_r_joint_inter: type fixed -> continuous
- joint shldr_f_l_joint_inter: type fixed -> continuous
- joint shldr_f_r_joint_inter: type fixed -> continuous
